Commit message: adding both the hands , bugs are there

File: urdf/mrm.xacro (robot description, xacro)
@@ -12,9 +12,9 @@
               iyy="170.667" iyz="0"
               izz="170.667"
-              size="1 1 1" />
+              size="1 1 3" />
   <m_joint name="${link_00_name}__${link_01_name}" type="revolute"
            axis_xyz="0 0 1"
-           origin_rpy="0 0 0" origin_xyz="0 0 0.5"
-           parent="base_link" child="link_01"
+           origin_rpy="105 0 0" origin_xyz="0 0.5 0.7"
+           parent="${link_00_name}" child="${link_01_name}"
            limit_e="1000" limit_l="-3.14" limit_u="3.14" limit_v="0.5" />
   <m_link_cylinder name="${link_01_name}"
@@ -29,5 +29,5 @@
            origin_rpy="0 0 0" origin_xyz="0 0 0.4"
            parent="link_01" child="link_02"
-           limit_e="1000" limit_l="0" limit_u="0.5" limit_v="0.5" />
+           limit_e="5000" limit_l="0" limit_u="1.0" limit_v="0.5" />
   <m_link_cylinder name="${link_02_name}"
               origin_rpy="0 0 0" origin_xyz="0 0 0.4"
@@ -41,5 +41,5 @@
            origin_rpy="0 0 0" origin_xyz="0 0 0.8"
            parent="link_02" child="link_03"
-           limit_e="1000" limit_l="0" limit_u="0.75" limit_v="0.5" />
+           limit_e="5000" limit_l="0" limit_u="1.3" limit_v="0.5" />
   <m_link_cylinder name="${link_03_name}"
               origin_rpy="0 0 0" origin_xyz="0 0 0.4"
@@ -53,5 +53,5 @@
            origin_rpy="0 0 0" origin_xyz="0 0 0.8"
            parent="link_03" child="link_04"
-           limit_e="1000" limit_l="0" limit_u="0.75" limit_v="0.5" />
+           limit_e="5000" limit_l="0" limit_u="1.5" limit_v="0.5" />
   <m_link_cylinder name="${link_04_name}"
               origin_rpy="0 0 0" origin_xyz="0 0 0.4"
@@ -65,7 +65,224 @@
            origin_rpy="0 0 0" origin_xyz="0 0 0.8"
            parent="link_04" child="link_05"
-           limit_e="1000" limit_l="-3.14" limit_u="3.14" limit_v="0.5" />
+           limit_e="5000" limit_l="-3.14" limit_u="3.14" limit_v="0.5" />
   <m_link_cylinder name="${link_05_name}"
               origin_rpy="0 0 0" origin_xyz="0 0 0.125"
+              mass="18.056"
+              ixx="0.479" ixy="0" ixz="0"
+              iyy="0.479" iyz="0"
+              izz="0.204"
+              radius="0.15" length="0.25" />
+   <joint name="gripper_extension" type="fixed">
+      <parent link="${link_05_name}"/>
+      <child link="gripper_pole"/>
+      <limit effort="1000.0" lower="-0.38" upper="0" velocity="0.5"/>
+     <origin rpy="0 0 0" xyz="0.15 0 0.2"/>
+   </joint>
+    <link name="gripper_pole">
+      <visual>
+        <geometry>
+          <cylinder length="0.6" radius="0.01"/>
+        </geometry>
+        <origin rpy="0 0 0 " xyz="-0.15 0 0.3"/>
+      </visual>
+     </link>
+  <joint name="left_gripper_joint" type="revolute">
+    <axis xyz="0 0 1"/>
+    <limit effort="1000.0" lower="0.0" upper="0.548" velocity="0.5"/>
+    <origin rpy="0 0 0" xyz="-0.15 0.01 0.6"/>
+    <parent link="gripper_pole"/>
+    <child link="left_gripper"/>
+  </joint>
+  <link name="left_gripper">
+    <visual>
+      <origin rpy="0.0 0 0" xyz="0 0 0"/>
+      <geometry>
+        <mesh filename="package://urdf_tutorial/meshes/l_finger.dae"/>
+      </geometry>
+    </visual>
+  </link>
+  <joint name="left_tip_joint" type="fixed">
+    <parent link="left_gripper"/>
+    <child link="left_tip"/>
+  </joint>
+  <link name="left_tip">
+    <visual>
+      <origin rpy="0.0 0 0" xyz="0.09137 0.00495 0"/>
+      <geometry>
+        <mesh filename="package://urdf_tutorial/meshes/l_finger_tip.dae"/>
+      </geometry>
+    </visual>
+  </link>
+  <joint name="right_gripper_joint" type="revolute">
+    <axis xyz="0 0 -1"/>
+    <limit effort="1000.0" lower="0.0" upper="0.548" velocity="0.5"/>
+    <origin rpy="0 0 0" xyz="-0.15 -0.01 0.60"/>
+    <parent link="gripper_pole"/>
+    <child link="right_gripper"/>
+  </joint>
+  <link name="right_gripper">
+    <visual>
+      <origin rpy="-3.1415 0 0" xyz="0 0 0"/>
+      <geometry>
+        <mesh filename="package://urdf_tutorial/meshes/l_finger.dae"/>
+      </geometry>
+    </visual>
+  </link>
+  <joint name="right_tip_joint" type="fixed">
+    <parent link="right_gripper"/>
+    <child link="right_tip"/>
+  </joint>
+  <link name="right_tip">
+    <visual>
+      <origin rpy="-3.1415 0 0" xyz="0.09137 0.00495 0"/>
+      <geometry>
+        <mesh filename="package://urdf_tutorial/meshes/l_finger_tip.dae"/>
+      </geometry>
+    </visual>
+  </link>
+  <link name="right_base">
+    <visual>
+      <geometry>
+        <box size="1 0.1 0.1"/>
+      </geometry>
+      <material name="white"/>
+      <origin xyz="0 -0.4 -1.5"/>
+    </visual>
+  </link>
+  <joint name="right_base_joint" type="fixed">
+    <parent link="base_link"/>
+    <child link="right_base"/>
+    <origin xyz="0 0 -0.05"/>
+  </joint>
+  <link name="right_front_wheel">
+    <visual>
+      <origin rpy="1.57075 0 0" xyz="0 0 0"/>
+      <geometry>
+        <cylinder length="0.1" radius="0.035"/>
+      </geometry>
+      <material name="black"/>
+      <origin rpy="0 0 0" xyz="0 0 0"/>
+    </visual>
+  </link>
+  <joint name="right_front_wheel_joint" type="continuous">
+    <axis rpy="0 0 0" xyz="0 3 0"/>
+    <parent link="right_base"/>
+    <child link="right_front_wheel"/>
+    <origin rpy="0 0 0" xyz="0.45 -0.4 -1.55"/>
+  </joint>
+  <link name="right_back_wheel">
+    <visual>
+      <origin rpy="1.57075 0 0" xyz="0 0 0"/>
+      <geometry>
+        <cylinder length="0.1" radius="0.035"/>
+      </geometry>
+      <material name="black"/>
+    </visual>
+  </link>
+  <joint name="right_back_wheel_joint" type="continuous">
+    <axis rpy="0 0 0" xyz="0 3 0"/>
+    <parent link="right_base"/>
+    <child link="right_back_wheel"/>
+    <origin rpy="0 0 0" xyz="-0.45 -0.4 -1.55"/>
+  </joint>
+  <link name="left_base">
+    <visual>
+      <geometry>
+        <box size="1 0.1 0.1"/>
+      </geometry>
+      <material name="white"/>
+      <origin xyz="0 0.4 -1.5"/>
+    </visual>
+  </link>
+  <joint name="left_base_joint" type="fixed">
+    <parent link="base_link"/>
+    <child link="left_base"/>
+    <origin xyz="0 0 -0.05"/>
+  </joint>
+<link name="left_front_wheel">
+    <visual>
+      <origin rpy="1.57075 0 0" xyz="0 0 0"/>
+      <geometry>
+        <cylinder length="0.1" radius="0.035"/>
+      </geometry>
+      <material name="black"/>
+    </visual>
+  </link>
+  <joint name="left_front_wheel_joint" type="continuous">
+    <axis rpy="0 0 0" xyz="0 3 0"/>
+    <parent link="left_base"/>
+    <child link="left_front_wheel"/>0.38 0.1
+    <origin rpy="0 0 0" xyz="0.45 0.4 -1.55"/>
+  </joint>
+<link name="left_back_wheel">
+    <visual>
+      <origin rpy="1.57075 0 0" xyz="0 0 0"/>
+      <geometry>
+        <cylinder length="0.1" radius="0.035"/>
+      </geometry>
+      <material name="black"/>
+    </visual>
+  </link>
+  <joint name="left_back_wheel_joint" type="continuous">
+    <axis rpy="0 0 0" xyz="0 3 0"/>
+    <parent link="left_base"/>
+    <child link="left_back_wheel"/>
+    <origin rpy="0 0 0" xyz="-0.45 0.4 -1.55"/>
+  </joint>
+<m_joint name="${link_00_name}__${left_joint}" type="revolute"
+           axis_xyz="0 0 1"
+           origin_rpy="105 0 0" origin_xyz="0 -0.5 0.7"
+           parent="${link_00_name}" child="${left_joint}"
+           limit_e="1000" limit_l="-3.14" limit_u="3.14" limit_v="0.5" />
+  <m_link_cylinder name="${left_joint}"
+              origin_rpy="0 0 0" origin_xyz="0 0 -0.2"
+              mass="157.633"
+              ixx="13.235" ixy="0" ixz="0"
+              iyy="13.235" iyz="0"
+              izz="9.655"
+              length="0.4" radius="0.35" />
+<m_joint name="${left_joint}__${cylinder_1}" type="revolute"
+           axis_xyz="0 1 0"
+           origin_rpy="0 0 0" origin_xyz="0 0 -0.4"
+           parent="left_joint" child="cylinder_1"
+           limit_e="5000" limit_l="0" limit_u="1.0" limit_v="0.5" />
+  <m_link_cylinder name="${cylinder_1}"
+              origin_rpy="0 0 0" origin_xyz="0 0 -0.4"
+              mass="57.906"
+              ixx="12.679" ixy="0" ixz="0"
+              iyy="12.679" iyz="0"
+              izz="0.651"
+              radius="0.15" length="0.8" />
+<m_joint name="${cylinder_1}__${cylinder2}" type="revolute"
+           axis_xyz="0 1 0"
+           origin_rpy="0 0 0" origin_xyz="0 0 -0.8"
+           parent="cylinder_1" child="cylinder2"
+           limit_e="5000" limit_l="0" limit_u="1.3" limit_v="0.5" />
+  <m_link_cylinder name="${cylinder2}"
+              origin_rpy="0 0 0" origin_xyz="0 0 -0.4"
+              mass="57.906"
+              ixx="12.679" ixy="0" ixz="0"
+              iyy="12.679" iyz="0"
+              izz="0.651"
+              radius="0.15" length="0.8" />
+  <m_joint name="${cylinder2}__${cylinder3}" type="revolute"
+           axis_xyz="0 1 0"
+           origin_rpy="0 0 0" origin_xyz="0 0 -0.8"
+           parent="cylinder2" child="cylinder3"
+           limit_e="5000" limit_l="0" limit_u="1.5" limit_v="0.5" />
+  <m_link_cylinder name="${cylinder3}"
+              origin_rpy="0 0 0" origin_xyz="0 0 -0.4"
+              mass="57.906"
+              ixx="12.679" ixy="0" ixz="0"
+              iyy="12.679" iyz="0"
+              izz="0.651"
+              radius="0.15" length="0.8" />
+  <m_joint name="${cylinder3}__${cylinder4}" type="revolute"
+           axis_xyz="0 0 1"
+           origin_rpy="0 0 0" origin_xyz="0 0 -0.8"
+           parent="cylinder3" child="cylinder4"
+           limit_e="5000" limit_l="-3.14" limit_u="3.14" limit_v="0.5" />
+  <m_link_cylinder name="${cylinder4}"
+              origin_rpy="0 0 0" origin_xyz="0 0 -0.125"
               mass="18.056"
               ixx="0.479" ixy="0" ixz="0"

File: urdf/robot_parameters.xacro (robot description, xacro)
@@ -7,3 +7,8 @@
   <xacro:property name="link_04_name" value="link_04" />
   <xacro:property name="link_05_name" value="link_05" />
+  <xacro:property name="left_joint" value="left_joint" />
+  <xacro:property name="cylinder_1" value="cylinder_1" />
+  <xacro:property name="cylinder2" value="cylinder2" />
+  <xacro:property name="cylinder3" value="cylinder3" />
+  <xacro:property name="cylinder4" value="cylinder4" />
 </robot>

Commit message: changed joints links name as parameters

File: urdf/mrm.xacro (robot description, xacro)
@@ -6,14 +6,14 @@
   <!-- END - Include -->
   <!-- BGN - Robot description -->
-  <m_link_box name="${link_00_name}"
+  <m_link_cylinder name="${link_00_name}"
               origin_rpy="0 0 0" origin_xyz="0 0 0"
-              mass="1024"
-              ixx="170.667" ixy="0" ixz="0"
-              iyy="170.667" iyz="0"
-              izz="170.667"
-              size="1 1 3" />
+              mass="10240"
+              ixx="1700.667" ixy="0" ixz="0"
+              iyy="1700.667" iyz="0"
+              izz="1700.667"
+              length="4" radius="0.5" />
   <m_joint name="${link_00_name}__${link_01_name}" type="revolute"
            axis_xyz="0 0 1"
-           origin_rpy="-1.57 0 0" origin_xyz="0 0.5 0.7"
+           origin_rpy="-1.57 0 0" origin_xyz="0 0.5 1.5"
            parent="${link_00_name}" child="${link_01_name}"
            limit_e="1000" limit_l="-3.14" limit_u="3.14" limit_v="0.5" />
@@ -141,99 +141,10 @@
     </visual>
   </link>
-  <link name="right_base">
-    <visual>
-      <geometry>
-        <box size="1 0.1 0.1"/>
-      </geometry>
-      <material name="white"/>
-      <origin xyz="0 -0.4 -1.5"/>
-    </visual>
-  </link>
-  <joint name="right_base_joint" type="fixed">
-    <parent link="base_link"/>
-    <child link="right_base"/>
-    <origin xyz="0 0 -0.05"/>
-  </joint>
-  <link name="right_front_wheel">
-    <visual>
-      <origin rpy="1.57075 0 0" xyz="0 0 0"/>
-      <geometry>
-        <cylinder length="0.1" radius="0.035"/>
-      </geometry>
-      <material name="black"/>
-      <origin rpy="0 0 0" xyz="0 0 0"/>
-    </visual>
-  </link>
-  <joint name="right_front_wheel_joint" type="continuous">
-    <axis rpy="0 0 0" xyz="0 3 0"/>
-    <parent link="right_base"/>
-    <child link="right_front_wheel"/>
-    <origin rpy="0 0 0" xyz="0.45 -0.4 -1.55"/>
-  </joint>
-  <link name="right_back_wheel">
-    <visual>
-      <origin rpy="1.57075 0 0" xyz="0 0 0"/>
-      <geometry>
-        <cylinder length="0.1" radius="0.035"/>
-      </geometry>
-      <material name="black"/>
-    </visual>
-  </link>
-  <joint name="right_back_wheel_joint" type="continuous">
-    <axis rpy="0 0 0" xyz="0 3 0"/>
-    <parent link="right_base"/>
-    <child link="right_back_wheel"/>
-    <origin rpy="0 0 0" xyz="-0.45 -0.4 -1.55"/>
-  </joint>
-  <link name="left_base">
-    <visual>
-      <geometry>
-        <box size="1 0.1 0.1"/>
-      </geometry>
-      <material name="white"/>
-      <origin xyz="0 0.4 -1.5"/>
-    </visual>
-  </link>
-  <joint name="left_base_joint" type="fixed">
-    <parent link="base_link"/>
-    <child link="left_base"/>
-    <origin xyz="0 0 -0.05"/>
-  </joint>
-<link name="left_front_wheel">
-    <visual>
-      <origin rpy="1.57075 0 0" xyz="0 0 0"/>
-      <geometry>
-        <cylinder length="0.1" radius="0.035"/>
-      </geometry>
-      <material name="black"/>
-    </visual>
-  </link>
-  <joint name="left_front_wheel_joint" type="continuous">
-    <axis rpy="0 0 0" xyz="0 3 0"/>
-    <parent link="left_base"/>
-    <child link="left_front_wheel"/>0.38 0.1
-    <origin rpy="0 0 0" xyz="0.45 0.4 -1.55"/>
-  </joint>
-<link name="left_back_wheel">
-    <visual>
-      <origin rpy="1.57075 0 0" xyz="0 0 0"/>
-      <geometry>
-        <cylinder length="0.1" radius="0.035"/>
-      </geometry>
-      <material name="black"/>
-    </visual>
-  </link>
-  <joint name="left_back_wheel_joint" type="continuous">
-    <axis rpy="0 0 0" xyz="0 3 0"/>
-    <parent link="left_base"/>
-    <child link="left_back_wheel"/>
-    <origin rpy="0 0 0" xyz="-0.45 0.4 -1.55"/>
-  </joint>
-<m_joint name="${link_00_name}__${left_joint}" type="revolute"
+<m_joint name="${link_00_name}__${link_11_name}" type="revolute"
            axis_xyz="0 0 1"
            origin_rpy="-1.57 0 0" origin_xyz="0 -0.5 0.7"
-           parent="${link_00_name}" child="${left_joint}"
+           parent="${link_00_name}" child="${link_11_name}"
            limit_e="1000" limit_l="-3.14" limit_u="3.14" limit_v="0.5" />
-  <m_link_cylinder name="${left_joint}"
+  <m_link_cylinder name="${link_11_name}"
               origin_rpy="0 0 0" origin_xyz="0 0 -0.2"
               mass="157.633"
@@ -242,10 +153,10 @@
               izz="9.655"
               length="0.4" radius="0.35" />
-<m_joint name="${left_joint}__${cylinder_1}" type="revolute"
+<m_joint name="${link_11_name}__${link_12_name}" type="revolute"
            axis_xyz="0 1 0"
            origin_rpy="0 0 0" origin_xyz="0 0 -0.4"
-           parent="left_joint" child="cylinder_1"
+           parent="${link_11_name}" child="${link_12_name}"
            limit_e="5000" limit_l="0" limit_u="1.0" limit_v="0.5" />
-  <m_link_cylinder name="${cylinder_1}"
+  <m_link_cylinder name="${link_12_name}"
               origin_rpy="0 0 0" origin_xyz="0 0 -0.4"
               mass="57.906"
@@ -254,10 +165,10 @@
               izz="0.651"
               radius="0.15" length="0.8" />
-<m_joint name="${cylinder_1}__${cylinder2}" type="revolute"
+<m_joint name="${link_12_name}__${link_13_name}" type="revolute"
            axis_xyz="0 1 0"
            origin_rpy="0 0 0" origin_xyz="0 0 -0.8"
-           parent="cylinder_1" child="cylinder2"
+           parent="${link_12_name}" child="${link_13_name}"
            limit_e="5000" limit_l="0" limit_u="1.3" limit_v="0.5" />
-  <m_link_cylinder name="${cylinder2}"
+  <m_link_cylinder name="${link_13_name}"
               origin_rpy="0 0 0" origin_xyz="0 0 -0.4"
               mass="57.906"
@@ -266,10 +177,10 @@
               izz="0.651"
               radius="0.15" length="0.8" />
-  <m_joint name="${cylinder2}__${cylinder3}" type="revolute"
+  <m_joint name="${link_13_name}__${link_14_name}" type="revolute"
            axis_xyz="0 1 0"
            origin_rpy="0 0 0" origin_xyz="0 0 -0.8"
-           parent="cylinder2" child="cylinder3"
+           parent="${link_13_name}" child="${link_14_name}"
            limit_e="5000" limit_l="0" limit_u="1.5" limit_v="0.5" />
-  <m_link_cylinder name="${cylinder3}"
+  <m_link_cylinder name="${link_14_name}"
               origin_rpy="0 0 0" origin_xyz="0 0 -0.4"
               mass="57.906"
@@ -278,10 +189,10 @@
               izz="0.651"
               radius="0.15" length="0.8" />
-  <m_joint name="${cylinder3}__${cylinder4}" type="revolute"
+  <m_joint name="${link_14_name}__${link_15_name}" type="revolute"
            axis_xyz="0 0 1"
            origin_rpy="0 0 0" origin_xyz="0 0 -0.8"
-           parent="cylinder3" child="cylinder4"
+           parent="${link_14_name}" child="${link_15_name}"
            limit_e="5000" limit_l="-3.14" limit_u="3.14" limit_v="0.5" />
-  <m_link_cylinder name="${cylinder4}"
+  <m_link_cylinder name="${link_15_name}"
               origin_rpy="0 0 0" origin_xyz="0 0 -0.125"
               mass="18.056"

File: urdf/robot_parameters.xacro (robot description, xacro)
@@ -7,8 +7,13 @@
   <xacro:property name="link_04_name" value="link_04" />
   <xacro:property name="link_05_name" value="link_05" />
-  <xacro:property name="left_joint" value="left_joint" />
-  <xacro:property name="cylinder_1" value="cylinder_1" />
+  <!-- <xacro:property name="link_11_name" value="link_11" /> -->
+  <!-- <xacro:property name="cylinder_1" value="cylinder_1" />
   <xacro:property name="cylinder2" value="cylinder2" />
   <xacro:property name="cylinder3" value="cylinder3" />
-  <xacro:property name="cylinder4" value="cylinder4" />
+  <xacro:property name="cylinder4" value="cylinder4" /> -->
+  <xacro:property name="link_11_name" value="link_11" />
+  <xacro:property name="link_12_name" value="link_12" />
+  <xacro:property name="link_13_name" value="link_13" />
+  <xacro:property name="link_14_name" value="link_14" />
+  <xacro:property name="link_15_name" value="link_15" />
 </robot>

Commit message: removed gripper codes

File: urdf/mrm.xacro (robot description, xacro)
@@ -73,72 +73,4 @@
               izz="0.564"
               radius="0.05" length="0.25" />
-   <joint name="gripper_extension" type="fixed">
-      <parent link="${link_05_name}"/>
-      <child link="gripper_pole"/>
-      <limit effort="1000.0" lower="-0.38" upper="0" velocity="0.5"/>
-     <origin rpy="0 0 0" xyz="0.15 0 0.2"/>
-   </joint>
-    <link name="gripper_pole">
-      <visual>
-        <geometry>
-          <cylinder length="0.6" radius="0.01"/>
-        </geometry>
-        <origin rpy="0 0 0 " xyz="-0.15 0 0.3"/>
-      </visual>
-     </link>
-  <joint name="left_gripper_joint" type="revolute">
-    <axis xyz="0 0 1"/>
-    <limit effort="1000.0" lower="0.0" upper="0.548" velocity="0.5"/>
-    <origin rpy="0 0 0" xyz="-0.15 0.01 0.6"/>
-    <parent link="gripper_pole"/>
-    <child link="left_gripper"/>
-  </joint>
-  <link name="left_gripper">
-    <visual>
-      <origin rpy="0.0 0 0" xyz="0 0 0"/>
-      <geometry>
-        <mesh filename="package://urdf_tutorial/meshes/l_finger.dae"/>
-      </geometry>
-    </visual>
-  </link>
-  <joint name="left_tip_joint" type="fixed">
-    <parent link="left_gripper"/>
-    <child link="left_tip"/>
-  </joint>
-  <link name="left_tip">
-    <visual>
-      <origin rpy="0.0 0 0" xyz="0.09137 0.00495 0"/>
-      <geometry>
-        <mesh filename="package://urdf_tutorial/meshes/l_finger_tip.dae"/>
-      </geometry>
-    </visual>
-  </link>
-  <joint name="right_gripper_joint" type="revolute">
-    <axis xyz="0 0 -1"/>
-    <limit effort="1000.0" lower="0.0" upper="0.548" velocity="0.5"/>
-    <origin rpy="0 0 0" xyz="-0.15 -0.01 0.60"/>
-    <parent link="gripper_pole"/>
-    <child link="right_gripper"/>
-  </joint>
-  <link name="right_gripper">
-    <visual>
-      <origin rpy="-3.1415 0 0" xyz="0 0 0"/>
-      <geometry>
-        <mesh filename="package://urdf_tutorial/meshes/l_finger.dae"/>
-      </geometry>
-    </visual>
-  </link>
-  <joint name="right_tip_joint" type="fixed">
-    <parent link="right_gripper"/>
-    <child link="right_tip"/>
-  </joint>
-  <link name="right_tip">
-    <visual>
-      <origin rpy="-3.1415 0 0" xyz="0.09137 0.00495 0"/>
-      <geometry>
-        <mesh filename="package://urdf_tutorial/meshes/l_finger_tip.dae"/>
-      </geometry>
-    </visual>
-  </link>
 <m_joint name="${link_00_name}__${link_11_name}" type="revolute"
            axis_xyz="0 0 1"

Commit message: added left hand gripper

File: urdf/mrm.xacro (robot description, xacro)
@@ -73,4 +73,59 @@
               izz="0.564"
               radius="0.05" length="0.25" />
+  <!-- adding gripper here -->
+  <joint name="left_gripper_joint" type="revolute">
+    <axis xyz="0 0 1" />
+    <limit effort="1000.0" lower="0.0" upper="0.548" velocity="0.5" />
+    <origin rpy="-1.57 0 0" xyz="0.0 0.0 0.25" />
+    <parent link="${link_05_name}" />
+    <child link="left_gripper" />
+  </joint>
+  <link name="left_gripper">
+    <visual>
+      <origin rpy="0.0 0 0" xyz="0 0 0" />
+      <geometry>
+        <mesh filename="package://mrm_description/meshes/l_finger.dae" scale="${scale_value} ${scale_value} ${scale_value} "/>
+      </geometry>
+    </visual>
+  </link>
+  <joint name="left_tip_joint" type="fixed">
+    <parent link="left_gripper" />
+    <child link="left_tip" />
+  </joint>
+  <link name="left_tip">
+    <visual>
+      <origin rpy="0.0 0 0" xyz="0.09137 0.00495 0" />
+      <geometry>
+        <mesh filename="package://mrm_description/meshes/l_finger_tip.dae" scale="${scale_value} ${scale_value} ${scale_value} " />
+      </geometry>
+    </visual>
+  </link>
+  <joint name="right_gripper_joint" type="revolute">
+    <axis xyz="0 0 -1" />
+    <limit effort="1000.0" lower="0.0" upper="0.548" velocity="0.5" />
+    <origin rpy="-1.57 0 0" xyz="0.0 0.0 0.25" />
+    <parent link="${link_05_name}" />
+    <child link="right_gripper" />
+  </joint>
+  <link name="right_gripper">
+    <visual>
+      <origin rpy="-3.1415 0 0" xyz="0 0 0" />
+      <geometry>
+        <mesh filename="package://mrm_description/meshes/l_finger.dae" scale="${scale_value} ${scale_value} ${scale_value} " />
+      </geometry>
+    </visual>
+  </link>
+  <joint name="right_tip_joint" type="fixed">
+    <parent link="right_gripper" />
+    <child link="right_tip" />
+  </joint>
+  <link name="right_tip">
+    <visual>
+      <origin rpy="-3.1415 0 0" xyz="0.09137 0.00495 0" />
+      <geometry>
+        <mesh filename="package://mrm_description/meshes/l_finger_tip.dae" scale="${scale_value} ${scale_value} ${scale_value} "/>
+      </geometry>
+    </visual>
+  </link>
 <m_joint name="${link_00_name}__${link_11_name}" type="revolute"
            axis_xyz="0 0 1"

File: urdf/robot_parameters.xacro (robot description, xacro)
@@ -17,3 +17,4 @@
   <xacro:property name="link_14_name" value="link_14" />
   <xacro:property name="link_15_name" value="link_15" />
+  <xacro:property name="scale_value" value="5" />
 </robot>
