Commit message: added camera and other files

File: urdf/mrm.xacro (robot description, xacro)
@@ -439,6 +439,6 @@
 <!-- addding camera -->
 <joint name="camera_joint" type="fixed">
-  <axis xyz="0 1 0" />
-  <origin xyz="0 0 4.1" rpy="0 0 0"/>
+  <axis xyz="0 0 0" />
+  <origin xyz="0 0 4.5" rpy="0 0 0"/>
   <parent link="base_link"/>
   <child link="camera_link"/>
@@ -494,18 +494,8 @@
     </plugin>
 </gazebo>
-<joint name="camera_optical_joint" type="fixed">
-  <!-- these values have to be these values otherwise the gazebo camera
-      image won't be aligned properly with the frame it is supposedly
-      originating from -->
-  <origin xyz="0 0 0" rpy="${-pi/2} 0 ${-pi/2}"/>
-  <parent link="camera_link"/>
-  <child link="camera_link_optical"/>
-</joint>
-<link name="camera_link_optical">
-</link>
-<gazebo reference="camera_link">
+<!-- <gazebo reference="camera_link">
   <sensor type="camera" name="camera1">
     <update_rate>30.0</update_rate>
-    <camera name="head">
+    <camera name="kinetic_camera">
       <horizontal_fov>1.3962634</horizontal_fov>
       <image>
@@ -530,5 +520,5 @@
       <imageTopicName>farming_robot/image_raw</imageTopicName>
       <cameraInfoTopicName>camera_info</cameraInfoTopicName>
-      <frameName>camera_link_optical</frameName>
+      <frameName>camera_link</frameName>
       <hackBaseline>0.07</hackBaseline>
       <distortionK1>0.0</distortionK1>
@@ -539,4 +529,46 @@
     </plugin>
   </sensor>
+</gazebo> -->
+<gazebo reference="camera_link">
+  <sensor name="camera_link_camera" type="depth">
+    <update_rate>20</update_rate>
+    <camera>
+      <!-- <horizontal_fov>1.047198</horizontal_fov> -->
+      <horizontal_fov>2.0</horizontal_fov>
+      <image>
+        <width>640</width>
+        <height>480</height>
+        <format>R8G8B8</format>
+      </image>
+      <clip>
+        <near>0.05</near>
+        <far>6</far>
+      </clip>
+    </camera>
+    <plugin name="camera_link_controller" filename="libgazebo_ros_openni_kinect.so">
+      <baseline>0.2</baseline>
+      <alwaysOn>true</alwaysOn>
+      <updateRate>1.0</updateRate>
+      <cameraName>${camera_name}_ir</cameraName>
+      <imageTopicName>/${camera_name}/color/image_raw</imageTopicName>
+      <cameraInfoTopicName>/${camera_name}/color/camera_info</cameraInfoTopicName>
+      <depthImageTopicName>/${camera_name}/depth/image_raw</depthImageTopicName>
+      <depthImageInfoTopicName>/${camera_name}/depth/camera_info</depthImageInfoTopicName>
+      <pointCloudTopicName>/${camera_name}/depth/points</pointCloudTopicName>
+      <frameName>${frame_name}</frameName>
+      <pointCloudCutoff>0.5</pointCloudCutoff>
+      <pointCloudCutoffMax>3.0</pointCloudCutoffMax>
+      <distortionK1>0.00000001</distortionK1>
+      <distortionK2>0.00000001</distortionK2>
+      <distortionK3>0.00000001</distortionK3>
+      <distortionT1>0.00000001</distortionT1>
+      <distortionT2>0.00000001</distortionT2>
+      <CxPrime>0</CxPrime>
+      <Cx>0</Cx>
+      <Cy>0</Cy>
+      <focalLength>0</focalLength>
+      <hackBaseline>0</hackBaseline>
+    </plugin>
+  </sensor>
 </gazebo>
 </robot>

File: urdf/robot_parameters.xacro (robot description, xacro)
@@ -18,3 +18,9 @@
   <xacro:property name="link_15_name" value="link_15" />
   <xacro:property name="scale_value" value="5" />
+  <xacro:property name="scale_value" value="5" />
+  <xacro:property name="effort_value" value="10000" />
+  <xacro:property name="camera_link" value="0.25" />
+  <xacro:property name="cam_color" value="Gazebo/Red" />
+  <xacro:property name="camera_name" value="kinnect" />
+  <xacro:property name="frame_name" value="camera_link" />
 </robot>

Commit message: added gripper to gazebo

File: urdf/mrm.xacro (robot description, xacro)
@@ -4,5 +4,10 @@
   <xacro:include filename="$(find mrm_description)/urdf/robot_parameters.xacro" />
   <xacro:include filename="$(find mrm_description)/urdf/links_joints.xacro" />
-  <!-- END - Include -->
+  <xacro:macro name="default_inertial" params="mass">
+    <inertial>
+      <mass value="${mass}" />
+      <inertia ixx="1.0" ixy="0.0" ixz="0.0" iyy="1.0" iyz="0.0" izz="1.0" />
+    </inertial>
+  </xacro:macro>  <!-- END - Include -->
   <!-- BGN - Robot description -->
   <m_link_cylinder name="${link_00_name}"
@@ -88,5 +93,15 @@
       </geometry>
     </visual>
-  </link>
+    <xacro:default_inertial mass="1"/>
+  </link>
+  <transmission name="top_left_gripper_joint_trans" type="SimpleTransmission">
+    <type>transmission_interface/SimpleTransmission</type>
+    <actuator name="top_left_gripper_joint_gripper_motor">
+      <mechanicalReduction>1</mechanicalReduction>
+    </actuator>
+    <joint name="top_left_gripper_joint">
+      <hardwareInterface>PositionJointInterface</hardwareInterface>
+    </joint>
+  </transmission>
   <joint name="top_left_tip_joint" type="fixed">
     <parent link="top_left_gripper" />
@@ -115,5 +130,15 @@
       </geometry>
     </visual>
-  </link>
+    <xacro:default_inertial mass="1"/>
+  </link>
+  <transmission name="down_left_gripper_joint_trans" type="SimpleTransmission">
+    <type>transmission_interface/SimpleTransmission</type>
+    <actuator name="down_left_gripper_joint_gripper_motor">
+      <mechanicalReduction>1</mechanicalReduction>
+    </actuator>
+    <joint name="down_left_gripper_joint">
+      <hardwareInterface>PositionJointInterface</hardwareInterface>
+    </joint>
+  </transmission>
   <joint name="down_left_tip_joint" type="fixed">
     <parent link="down_left_gripper" />
@@ -203,5 +228,15 @@
       </geometry>
     </visual>
-  </link>
+    <xacro:default_inertial mass="1"/>
+  </link>
+  <transmission name="top_right_gripper_joint_trans" type="SimpleTransmission">
+    <type>transmission_interface/SimpleTransmission</type>
+    <actuator name="top_right_gripper_joint_gripper_motor">
+      <mechanicalReduction>1</mechanicalReduction>
+    </actuator>
+    <joint name="top_right_gripper_joint">
+      <hardwareInterface>PositionJointInterface</hardwareInterface>
+    </joint>
+  </transmission>
   <joint name="top_right_tip_joint" type="fixed">
     <parent link="top_right_gripper" />
@@ -230,5 +265,15 @@
       </geometry>
     </visual>
-  </link>
+    <xacro:default_inertial mass="1"/>
+  </link>
+  <transmission name="down_right_gripper_joint_trans" type="SimpleTransmission">
+    <type>transmission_interface/SimpleTransmission</type>
+    <actuator name="down_right_gripper_joint_gripper_motor">
+      <mechanicalReduction>1</mechanicalReduction>
+    </actuator>
+    <joint name="down_right_gripper_joint">
+      <hardwareInterface>PositionJointInterface</hardwareInterface>
+    </joint>
+  </transmission>
   <joint name="down_right_tip_joint" type="fixed">
     <parent link="down_right_gripper" />
@@ -440,5 +485,5 @@
 <joint name="camera_joint" type="fixed">
   <axis xyz="0 0 0" />
-  <origin xyz="0 0 4.5" rpy="0 0 0"/>
+  <origin xyz="0 0 4.5" rpy="0 -1.57 0"/>
   <parent link="base_link"/>
   <child link="camera_link"/>

Commit message: added kinnect camera and fake controllers for gripper

File: urdf/mrm.xacro (robot description, xacro)
@@ -99,7 +99,8 @@
     <actuator name="top_left_gripper_joint_gripper_motor">
       <mechanicalReduction>1</mechanicalReduction>
+      <hardwareInterface>hardware_interface/EffortJointInterface</hardwareInterface>
     </actuator>
     <joint name="top_left_gripper_joint">
-      <hardwareInterface>PositionJointInterface</hardwareInterface>
+      <hardwareInterface>hardware_interface/EffortJointInterface</hardwareInterface>
     </joint>
   </transmission>
@@ -136,7 +137,8 @@
     <actuator name="down_left_gripper_joint_gripper_motor">
       <mechanicalReduction>1</mechanicalReduction>
+      <hardwareInterface>hardware_interface/EffortJointInterface</hardwareInterface>
     </actuator>
     <joint name="down_left_gripper_joint">
-      <hardwareInterface>PositionJointInterface</hardwareInterface>
+      <hardwareInterface>hardware_interface/EffortJointInterface</hardwareInterface>
     </joint>
   </transmission>
@@ -234,7 +236,8 @@
     <actuator name="top_right_gripper_joint_gripper_motor">
       <mechanicalReduction>1</mechanicalReduction>
+      <hardwareInterface>hardware_interface/EffortJointInterface</hardwareInterface>
     </actuator>
     <joint name="top_right_gripper_joint">
-      <hardwareInterface>PositionJointInterface</hardwareInterface>
+      <hardwareInterface>hardware_interface/EffortJointInterface</hardwareInterface>
     </joint>
   </transmission>
@@ -271,7 +274,8 @@
     <actuator name="down_right_gripper_joint_gripper_motor">
       <mechanicalReduction>1</mechanicalReduction>
+      <hardwareInterface>hardware_interface/EffortJointInterface</hardwareInterface>
     </actuator>
     <joint name="down_right_gripper_joint">
-      <hardwareInterface>PositionJointInterface</hardwareInterface>
+      <hardwareInterface>hardware_interface/EffortJointInterface</hardwareInterface>
     </joint>
   </transmission>
@@ -485,5 +489,5 @@
 <joint name="camera_joint" type="fixed">
   <axis xyz="0 0 0" />
-  <origin xyz="0 0 4.5" rpy="0 -1.57 0"/>
+  <origin xyz="0 0 4.2" rpy="0.0 0.0 0.0"/>
   <parent link="base_link"/>
   <child link="camera_link"/>
@@ -494,5 +498,5 @@
     <origin xyz="0 0 0" rpy="0 0 0"/>
     <geometry>
-  <box size="${camera_link} ${camera_link} ${camera_link}"/>
+      <mesh filename="package://mrm_description/meshes/kinect.dae" scale="${scale_value} ${scale_value} ${scale_value} " />
     </geometry>
   </collision>
@@ -500,7 +504,7 @@
     <origin xyz="0 0 0" rpy="0 0 0"/>
     <geometry>
-  <box size="${camera_link} ${camera_link} ${camera_link}"/>
-    </geometry>
-    <material name="red"/>
+      <mesh filename="package://mrm_description/meshes/kinect.dae" scale="${scale_value} ${scale_value} ${scale_value} " />
+    </geometry>
+    <!-- <material name="red"/> -->
   </visual>
   <inertial>
@@ -510,10 +514,10 @@
   </inertial>
 </link>
-<gazebo reference="camera_link">
+<!-- <gazebo reference="camera_link">
   <material>${cam_color}</material>
   <mu1>0.2</mu1>
   <mu2>0.2</mu2>
   <selfCollide>true</selfCollide>
-</gazebo>
+</gazebo> -->
   <!-- END - Robot description -->
   <gazebo>

Commit message: added basket and written control commands

File: urdf/mrm.xacro (robot description, xacro)
@@ -99,8 +99,8 @@
     <actuator name="top_left_gripper_joint_gripper_motor">
       <mechanicalReduction>1</mechanicalReduction>
-      <hardwareInterface>hardware_interface/EffortJointInterface</hardwareInterface>
+      <hardwareInterface>hardware_interface/PositionJointInterface</hardwareInterface>
     </actuator>
     <joint name="top_left_gripper_joint">
-      <hardwareInterface>hardware_interface/EffortJointInterface</hardwareInterface>
+      <hardwareInterface>hardware_interface/PositionJointInterface</hardwareInterface>
     </joint>
   </transmission>
@@ -137,8 +137,8 @@
     <actuator name="down_left_gripper_joint_gripper_motor">
       <mechanicalReduction>1</mechanicalReduction>
-      <hardwareInterface>hardware_interface/EffortJointInterface</hardwareInterface>
+      <hardwareInterface>hardware_interface/PositionJointInterface</hardwareInterface>
     </actuator>
     <joint name="down_left_gripper_joint">
-      <hardwareInterface>hardware_interface/EffortJointInterface</hardwareInterface>
+      <hardwareInterface>hardware_interface/PositionJointInterface</hardwareInterface>
     </joint>
   </transmission>
@@ -215,80 +215,20 @@
               izz="0.0564"
               radius="0.05" length="0.25" />
-    <!-- adding right gripper here save -->
-  <joint name="top_right_gripper_joint" type="revolute">
+    <!-- adding basket -->
+  <joint name="basket_joint" type="fixed">
     <axis xyz="0 0 1" />
     <limit effort="1000.0" lower="0.0" upper="0.548" velocity="2.5" />
-    <origin rpy="0 0 0" xyz="0.0 0.0 -0.25" />
+    <origin rpy="0 -3.14, 0.0 " xyz="0.8 -0.3 0" />
     <parent link="${link_15_name}" />
-    <child link="top_right_gripper" />
-  </joint>
-  <link name="top_right_gripper">
+    <child link="basket_link" />
+  </joint>
+  <link name="basket_link">
     <visual>
       <origin rpy="0.0 0 0" xyz="0 0 0" />
       <geometry>
-        <mesh filename="package://mrm_description/meshes/l_finger.dae" scale="${scale_value} ${scale_value} ${scale_value} " />
+        <mesh filename="package://mrm_description/meshes/basket.dae" scale="${basket_scale} ${basket_scale} ${basket_scale} " />
       </geometry>
     </visual>
     <xacro:default_inertial mass="1"/>
-  </link>
-  <transmission name="top_right_gripper_joint_trans" type="SimpleTransmission">
-    <type>transmission_interface/SimpleTransmission</type>
-    <actuator name="top_right_gripper_joint_gripper_motor">
-      <mechanicalReduction>1</mechanicalReduction>
-      <hardwareInterface>hardware_interface/EffortJointInterface</hardwareInterface>
-    </actuator>
-    <joint name="top_right_gripper_joint">
-      <hardwareInterface>hardware_interface/EffortJointInterface</hardwareInterface>
-    </joint>
-  </transmission>
-  <joint name="top_right_tip_joint" type="fixed">
-    <parent link="top_right_gripper" />
-    <child link="top_right_tip" />
-  </joint>
-  <link name="top_right_tip">
-    <visual>
-      <origin rpy="0.0 0 0" xyz="0.09137 0.00495 0" />
-      <geometry>
-        <mesh filename="package://mrm_description/meshes/l_finger_tip.dae" scale="${scale_value} ${scale_value} ${scale_value} " />
-      </geometry>
-    </visual>
-  </link>
-  <joint name="down_right_gripper_joint" type="revolute">
-    <axis xyz="0 0 -1" />
-    <limit effort="1000.0" lower="0.0" upper="0.548" velocity="0.5" />
-    <origin rpy="0 0 0" xyz="0.0 0.0 -0.25" />
-    <parent link="${link_15_name}" />
-    <child link="down_right_gripper" />
-  </joint>
-  <link name="down_right_gripper">
-    <visual>
-      <origin rpy="-3.1415 0 0" xyz="0 0 0" />
-      <geometry>
-        <mesh filename="package://mrm_description/meshes/l_finger.dae" scale="${scale_value} ${scale_value} ${scale_value} " />
-      </geometry>
-    </visual>
-    <xacro:default_inertial mass="1"/>
-  </link>
-  <transmission name="down_right_gripper_joint_trans" type="SimpleTransmission">
-    <type>transmission_interface/SimpleTransmission</type>
-    <actuator name="down_right_gripper_joint_gripper_motor">
-      <mechanicalReduction>1</mechanicalReduction>
-      <hardwareInterface>hardware_interface/EffortJointInterface</hardwareInterface>
-    </actuator>
-    <joint name="down_right_gripper_joint">
-      <hardwareInterface>hardware_interface/EffortJointInterface</hardwareInterface>
-    </joint>
-  </transmission>
-  <joint name="down_right_tip_joint" type="fixed">
-    <parent link="down_right_gripper" />
-    <child link="down_right_tip" />
-  </joint>
-  <link name="down_right_tip">
-    <visual>
-      <origin rpy="-3.1415 0 0" xyz="0.09137 0.00495 0" />
-      <geometry>
-        <mesh filename="package://mrm_description/meshes/l_finger_tip.dae" scale="${scale_value} ${scale_value} ${scale_value} " />
-      </geometry>
-    </visual>
   </link>
   <!-- adding wheels -->

File: urdf/robot_parameters.xacro (robot description, xacro)
@@ -18,5 +18,5 @@
   <xacro:property name="link_15_name" value="link_15" />
   <xacro:property name="scale_value" value="5" />
-  <xacro:property name="scale_value" value="5" />
+  <xacro:property name="basket_scale" value="0.015" />
   <xacro:property name="effort_value" value="10000" />
   <xacro:property name="camera_link" value="0.25" />

Commit message: latest

File: urdf/mrm.xacro (robot description, xacro)
@@ -46,5 +46,5 @@
            origin_rpy="0 0 0" origin_xyz="0 0 0.8"
            parent="link_02" child="link_03"
-           limit_e="5000" limit_l="0" limit_u="1.57" limit_v="2.5" />
+           limit_e="5000" limit_l="-1.57" limit_u="1.57" limit_v="2.5" />
   <m_link_cylinder name="${link_03_name}"
               origin_rpy="0 0 0" origin_xyz="0 0 0.4"
@@ -58,5 +58,5 @@
            origin_rpy="0 0 0" origin_xyz="0 0 0.8"
            parent="link_03" child="link_04"
-           limit_e="5000" limit_l="0" limit_u="1.57" limit_v="2.5" />
+           limit_e="5000" limit_l="-1.57" limit_u="1.57" limit_v="2.5" />
   <m_link_cylinder name="${link_04_name}"
               origin_rpy="0 0 0" origin_xyz="0 0 0.4"
@@ -81,6 +81,6 @@
   <joint name="top_left_gripper_joint" type="revolute">
     <axis xyz="0 0 1" />
-    <limit effort="1000.0" lower="0.0" upper="0.548" velocity="0.5" />
-    <origin rpy="0 0 0" xyz="0.0 0.0 0.25" />
+    <limit effort="10.0" lower="0.0" upper="1.57" velocity="2.5" />
+    <origin rpy="0 0 3.14" xyz="0.0 0.0 0.25" />
     <parent link="${link_05_name}" />
     <child link="top_left_gripper" />
@@ -93,5 +93,5 @@
       </geometry>
     </visual>
-    <xacro:default_inertial mass="1"/>
+    <xacro:default_inertial mass="0.05"/>
   </link>
   <transmission name="top_left_gripper_joint_trans" type="SimpleTransmission">
@@ -99,8 +99,8 @@
     <actuator name="top_left_gripper_joint_gripper_motor">
       <mechanicalReduction>1</mechanicalReduction>
-      <hardwareInterface>hardware_interface/PositionJointInterface</hardwareInterface>
-    </actuator>
+        <hardwareInterface>hardware_interface/EffortJointInterface</hardwareInterface>
+      </actuator>
     <joint name="top_left_gripper_joint">
-      <hardwareInterface>hardware_interface/PositionJointInterface</hardwareInterface>
+      <hardwareInterface>hardware_interface/EffortJointInterface</hardwareInterface>
     </joint>
   </transmission>
@@ -119,6 +119,6 @@
   <joint name="down_left_gripper_joint" type="revolute">
     <axis xyz="0 0 -1" />
-    <limit effort="1000.0" lower="0.0" upper="0.548" velocity="0.5" />
-    <origin rpy="0 0 0" xyz="0.0 0.0 0.25" />
+    <limit effort="10.0" lower="0.0" upper="1.57" velocity="2.5" />
+    <origin rpy="0 0 3.14" xyz="0.0 0.0 0.25" />
     <parent link="${link_05_name}" />
     <child link="down_left_gripper" />
@@ -131,5 +131,5 @@
       </geometry>
     </visual>
-    <xacro:default_inertial mass="1"/>
+    <xacro:default_inertial mass="0.05"/>
   </link>
   <transmission name="down_left_gripper_joint_trans" type="SimpleTransmission">
@@ -137,8 +137,8 @@
     <actuator name="down_left_gripper_joint_gripper_motor">
       <mechanicalReduction>1</mechanicalReduction>
-      <hardwareInterface>hardware_interface/PositionJointInterface</hardwareInterface>
+      <hardwareInterface>hardware_interface/EffortJointInterface</hardwareInterface>
     </actuator>
     <joint name="down_left_gripper_joint">
-      <hardwareInterface>hardware_interface/PositionJointInterface</hardwareInterface>
+      <hardwareInterface>hardware_interface/EffortJointInterface</hardwareInterface>
     </joint>
   </transmission>
@@ -219,5 +219,5 @@
     <axis xyz="0 0 1" />
     <limit effort="1000.0" lower="0.0" upper="0.548" velocity="2.5" />
-    <origin rpy="0 -3.14, 0.0 " xyz="0.8 -0.3 0" />
+    <origin rpy="0.0 -3.14 0.0" xyz="0.8 -0.3 0" />
     <parent link="${link_15_name}" />
     <child link="basket_link" />
