Commit message: change gripper controllers and solved tif to png issue.

File: urdf/mrm.xacro (robot description, xacro)
@@ -79,5 +79,5 @@
               radius="0.05" length="0.25" />
   <!-- adding leftgripper here -->
-  <joint name="top_left_gripper_joint" type="revolute">
+  <!-- <joint name="top_left_gripper_joint" type="revolute">
     <axis xyz="0 0 1" />
     <limit effort="10.0" lower="0.0" upper="1.57" velocity="2.5" />
@@ -155,4 +155,93 @@
     </visual>
   </link>
+-->
+<joint name="gripper_extension" type="prismatic">
+  <parent link="${link_05_name}"/>
+  <child link="gripper_pole"/>
+  <limit effort="1000.0" lower="-${width*2-.02}" upper="0" velocity="0.5"/>
+  <origin rpy="0 0 3.14" xyz="${width-0.25} 0 0.2"/>
+  <limit effort="30" velocity="0.2"/>
+  <dynamics damping="0.0" friction="0.0"/>
+</joint>
+<link name="gripper_pole">
+  <visual>
+    <geometry>
+      <cylinder length="${polelen}" radius="0.01"/>
+    </geometry>
+    <origin xyz="${polelen/2} 0 0" rpy="0 ${pi/2} 0 "/>
+  </visual>
+  <collision>
+    <geometry>
+      <cylinder length="${polelen}" radius="0.01"/>
+    </geometry>
+    <origin xyz="${polelen/2} 0 0" rpy="0 ${pi/2} 0 "/>
+  </collision>
+  <xacro:default_inertial mass="0.05"/>
+</link>
+<transmission name="gripper_extension_trans" type="SimpleTransmission">
+  <type>transmission_interface/SimpleTransmission</type>
+  <actuator name="gripper_extension_motor">
+    <mechanicalReduction>1</mechanicalReduction>
+  </actuator>
+  <joint name="gripper_extension">
+    <hardwareInterface>hardware_interface/PositionJointInterface</hardwareInterface>
+  </joint>
+</transmission>
+<xacro:macro name="gripper" params="prefix reflect">
+  <joint name="${prefix}_gripper_joint" type="revolute">
+    <axis xyz="0 0 ${reflect}"/>
+    <limit effort="1000.0" lower="0.0" upper="0.548" velocity="0.5"/>
+    <origin rpy="0 0 0" xyz="${polelen} ${reflect*0.01} 0"/>
+    <parent link="gripper_pole"/>
+    <child link="${prefix}_gripper"/>
+    <limit effort="30" velocity="1.0"/>
+    <dynamics damping="0.0" friction="0.0"/>
+  </joint>
+  <link name="${prefix}_gripper">
+    <visual>
+      <origin rpy="${(reflect-1)/2*pi} 0 0" xyz="0 0 0"/>
+      <geometry>
+        <mesh filename="package://mrm_description/meshes/l_finger.dae" scale="${scale_value} ${scale_value} ${scale_value} " />
+      </geometry>
+    </visual>
+    <collision>
+      <geometry>
+        <mesh filename="package://mrm_description/meshes/l_finger.dae" scale="${scale_value} ${scale_value} ${scale_value} "/>
+      </geometry>
+      <origin rpy="${(reflect-1)/2*pi} 0 0" xyz="0 0 0"/>
+    </collision>
+    <xacro:default_inertial mass="0.05"/>
+  </link>
+  <transmission name="${prefix}_gripper_trans" type="SimpleTransmission">
+    <type>transmission_interface/SimpleTransmission</type>
+    <actuator name="${prefix}_gripper_motor">
+      <mechanicalReduction>1</mechanicalReduction>
+    </actuator>
+    <joint name="${prefix}_gripper_joint">
+      <hardwareInterface>hardware_interface/PositionJointInterface</hardwareInterface>
+    </joint>
+  </transmission>
+  <joint name="${prefix}_tip_joint" type="fixed">
+    <parent link="${prefix}_gripper"/>
+    <child link="${prefix}_tip"/>
+  </joint>
+  <link name="${prefix}_tip">
+    <visual>
+      <origin rpy="${(reflect-1)/2*pi} 0 0" xyz="0.09137 0.00495 0"/>
+      <geometry>
+        <mesh filename="package://mrm_description/meshes/l_finger_tip.dae" scale="${scale_value} ${scale_value} ${scale_value} "/>
+      </geometry>
+    </visual>
+    <collision>
+      <geometry>
+        <mesh filename="package://mrm_description/meshes/l_finger_tip.dae" scale="${scale_value} ${scale_value} ${scale_value} "/>
+      </geometry>
+      <origin rpy="${(reflect-1)/2*pi} 0 0" xyz="0.09137 0.00495 0"/>
+    </collision>
+    <xacro:default_inertial mass="0.05"/>
+  </link>
+</xacro:macro>
+<xacro:gripper prefix="left" reflect="1" />
+<xacro:gripper prefix="right" reflect="-1" />
 <m_joint name="${link_00_name}__${link_11_name}" type="revolute"
            axis_xyz="0 0 1"

File: urdf/robot_parameters.xacro (robot description, xacro)
@@ -25,3 +25,10 @@
   <xacro:property name="frame_name" value="camera_link" />
   <xacro:property name="M_PI" value="3.14" />
+  <xacro:property name="width" value="0.2" />
+  <xacro:property name="leglen" value="0.6" />
+  <xacro:property name="polelen" value="0.08" />
+  <xacro:property name="bodylen" value="0.6" />
+  <xacro:property name="baselen" value="0.4" />
+  <xacro:property name="wheeldiam" value="0.07" />
+  <xacro:property name="pi" value="3.1415" />
 </robot>
